File: hardware/SimsBharath_DAQ.kicad_sch (KiCad schematic)
At the start: 0 parts

Commit message: completed the design
Other:
- sheet CONNECTORS ports: added USB_FS_D N, USB_FS_D P, USB_FS_VBUS; removed {USB_FS_VBUS USB_FS_DM USB_FS_DP}
- sheet MCU ports: added USB_FS_D N, USB_FS_D P, USB_FS_VBUS; removed {USB_FS_VBUS USB_FS_DM USB_FS_DP}
Changed lines of the file:
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@@
+		)
+	)
+	(wire
+		(pts
+			(xy 156.21 97.79) (xy 177.8 97.79)
+		)
+		(stroke
+			(width 0)
+			(type default)
 		)
 	)
@@
 	(bus
 		(pts
+			(xy 156.21 92.71) (xy 177.8 92.71)
+		)
+		(stroke
+			(width 0)
+			(type default)
+		)
+	)
+	(wire
+		(pts
+			(xy 156.21 127) (xy 177.8 127)
+		)
+		(stroke
+			(width 0)
+			(type default)
+		)
+	)
+	(wire
+		(pts
+			(xy 156.21 124.46) (xy 177.8 124.46)
+		)
+		(stroke
+			(width 0)
+			(type default)
+		)
+	)
+	(wire
+		(pts
+			(xy 156.21 109.22) (xy 177.8 109.22)
+		)
+		(stroke
+			(width 0)
+			(type default)
+		)
+	)
+	(bus
+		(pts
+			(xy 156.21 132.08) (xy 177.8 132.08)
+		)
+		(stroke
+			(width 0)
+			(type default)
+		)
+	)
+	(wire
+		(pts
+			(xy 156.21 57.15) (xy 177.8 57.15)
+		)
+		(stroke
+			(width 0)
+			(type default)
+		)
+	)
+	(wire
+		(pts
+			(xy 156.21 116.84) (xy 177.8 116.84)
+		)
+		(stroke
+			(width 0)
+			(type default)
+		)
+	)
+	(bus
+		(pts
+			(xy 156.21 69.85) (xy 177.8 69.85)
+		)
+		(stroke
+			(width 0)
+			(type default)
+		)
+	)
+	(bus
+		(pts
+			(xy 156.21 87.63) (xy 177.8 87.63)
+		)
+		(stroke
+			(width 0)
+			(type default)
+		)
+	)
+	(wire
+		(pts
 			(xy 156.21 95.25) (xy 177.8 95.25)
 		)
@@
 	(wire
 		(pts
-			(xy 156.21 127) (xy 177.8 127)
-		)
-		(stroke
-			(width 0)
-			(type default)
-		)
-	)
-	(wire
-		(pts
-			(xy 156.21 124.46) (xy 177.8 124.46)
-		)
-		(stroke
-			(width 0)
-			(type default)
-		)
-	)
-	(wire
-		(pts
-			(xy 156.21 109.22) (xy 177.8 109.22)
-		)
-		(stroke
-			(width 0)
-			(type default)
-		)
-	)
-	(bus
-		(pts
-			(xy 156.21 132.08) (xy 177.8 132.08)
-		)
-		(stroke
-			(width 0)
-			(type default)
-		)
-	)
-	(wire
-		(pts
-			(xy 156.21 57.15) (xy 177.8 57.15)
-		)
-		(stroke
-			(width 0)
-			(type default)
-		)
-	)
-	(wire
-		(pts
-			(xy 156.21 116.84) (xy 177.8 116.84)
-		)
-		(stroke
-			(width 0)
-			(type default)
-		)
-	)
-	(bus
-		(pts
-			(xy 156.21 69.85) (xy 177.8 69.85)
-		)
-		(stroke
-			(width 0)
-			(type default)
-		)
-	)
-	(bus
-		(pts
-			(xy 156.21 87.63) (xy 177.8 87.63)
-		)
-		(stroke
-			(width 0)
-			(type default)
-		)
-	)
-	(wire
-		(pts
 			(xy 156.21 114.3) (xy 177.8 114.3)
 		)
@@
 		)
 	)
-	(bus
-		(pts
-			(xy 156.21 92.71) (xy 177.8 92.71)
+	(wire
+		(pts
+			(xy 156.21 100.33) (xy 177.8 100.33)
 		)
 		(stroke
@@
 		)
 		(pin "{DAC0 DAC1}" bidirectional
-			(at 156.21 95.25 0)
+			(at 156.21 92.71 0)
 			(effects
 				(font
@@
 			)
 		)
-		(pin "{USB_FS_VBUS USB_FS_DM USB_FS_DP}" bidirectional
-			(at 156.21 92.71 0)
+		(pin "USB_FS_D N" bidirectional
+			(at 156.21 95.25 0)
+			(effects
+				(font
+					(size 1.27 1.27)
+				)
+				(justify right)
+			)
+		)
+		(pin "USB_FS_D P" bidirectional
+			(at 156.21 97.79 0)
+			(effects
+				(font
+					(size 1.27 1.27)
+				)
+				(justify right)
+			)
+		)
+		(pin "USB_FS_VBUS" bidirectional
+			(at 156.21 100.33 0)
 			(effects
 				(font
@@
 		)
 		(pin "{DAC0 DAC1}" bidirectional
-			(at 177.8 95.25 180)
+			(at 177.8 92.71 180)
 			(effects
 				(font
@@
 			)
 		)
-		(pin "{USB_FS_VBUS USB_FS_DM USB_FS_DP}" bidirectional
-			(at 177.8 92.71 180)
-			(effects
-				(font
+		(pin "USB_FS_D N" bidirectional
+			(at 177.8 95.25 180)
+			(effects
+				(font
+					(size 1.27 1.27)
+				)
+				(justify left)
+			)
+		)
+		(pin "USB_FS_D P" bidirectional
+			(at 177.8 97.79 180)
+			(effects
+				(font
+					(size 1.27 1.27)
+				)
+				(justify left)
+			)
+		)
+		(pin "USB_FS_VBUS" bidirectional
+			(at 177.8 100.33 180)
+			(effects
+				(font

Commit message: completed the design with perfect mechanics
Other:
- sheet CONNECTORS ports: added none; removed USB_FS_VBUS
- sheet MCU ports: added none; removed USB_FS_VBUS
Changed lines of the file:
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@@
-	(wire
-		(pts
-			(xy 156.21 100.33) (xy 177.8 100.33)
-		)
-		(stroke
-			(width 0)
-			(type default)
-		)
-	)
 	(wire
 		(pts
@@
 			)
 		)
-		(pin "USB_FS_VBUS" bidirectional
-			(at 156.21 100.33 0)
-			(effects
-				(font
-					(size 1.27 1.27)
-				)
-				(justify right)
-			)
-		)
 		(instances
 			(project "SimsBharath_DAQ"
@@
 			(effects
 				(font
-					(size 1.27 1.27)
-				)
-				(justify left)
-			)
-		)
-		(pin "USB_FS_VBUS" bidirectional
-			(at 177.8 100.33 180)
-			(effects
-				(font

Commit message: Final Updated design
Other:
- sheet CONNECTORS ports: added PWM0, PWM1, PWM2, PWM3, PWM4, PWM5; removed PWM1[0..1], PWM[0..3]
- sheet MCU ports: added PWM0, PWM1, PWM2, PWM3, PWM4, PWM5; removed PWM1[0..1], PWM[0..3]
