File: hardware/SimsBharath_DAQ_Connectors.kicad_sch (KiCad schematic)
At the start: 54 parts, among them IC3 LAN8742A-CZ-TR, J1 Conn_02x05_Odd_Even, J10 702471052, J11 702471052, J2 USB1030-GF-P-B-B, J3 702471052, J4 702471052, J5 702471052, J6 702471052, J7 702471052, J8 702471052, J9 1-406507-5, T1 H1102NL, Y2 XRCGB25M000F3A16R0

Commit message: updated
Parts:
- added C38, C39: 1uF, Murata:GRM18x, symbol Murata:GRM188R72A104KA35D
- added R36, R37: 20k, Murata:RESC1608X95N, symbol Murata:PRF18BC471QB5RB
- renumbered IC3 to U3, T1 to U4, Y2 to X2
Connections:
- net DAC0: now also R37.2; no longer J4.2
- net DAC1: now also R36.2; no longer J4.1
- net GND: now also C38.2, C39.2
- net TX P: now reaches J9.1, U4.16 (TX+)
- net TX N: now reaches J9.2, U4.14 (TX-)
- net RX P: now reaches J9.3, U4.11 (RX+)
- net RX N: now reaches J9.6, U4.9 (RX-)
- new net M_DAC0: C39.1, J4.1, R37.1
- new net M_DAC1: C38.1, J4.2, R36.1

Commit message: completed the design
Connections:
- net ADC3_1: now also J3.8; no longer J3.1
- net ADC3_2: now also J3.7; no longer J3.2
- net ADC3_3: now also J3.6; no longer J3.3
- net ADC3_4: now also J3.5; no longer J3.4
- net ADC3_5: now also J3.4; no longer J3.5
- net ADC3_6: now also J3.3; no longer J3.6
- net ADC3_7: now also J3.2; no longer J3.7
- net ADC3_8: now also J3.1; no longer J3.8
- net USB_FS_DM renamed USB_FS_D N
- net USB_FS_DP renamed USB_FS_D P

Commit message: completed the design with perfect mechanics
Parts:
- added J12: Conn_01x03, Connector_PinHeader_2.54mm:PinHeader_1x03_P2.54mm_Vertical, symbol Connector_Generic:Conn_01x03
Connections:
- net +3.3V: no longer J1.1 (Pin_1)
- net +5V: now also J12.2 (Pin_2)
- net USB_FS_VBUS renamed +5V-USB
- net +5V-USB: now also J12.3 (Pin_3)
- new net +5V-JTAG: J1.1 (Pin_1), J12.1 (Pin_1)
Changed lines of the file:
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@@
 		)
 	)
+	(wire
+		(pts
+			(xy 30.48 34.29) (xy 35.56 34.29)
+		)
+		(stroke
+			(width 0)
+			(type default)
+		)
+	)
 	(bus
 		(pts
@@
 	(wire
 		(pts
+			(xy 44.45 53.34) (xy 48.26 53.34)
+		)
+		(stroke
+			(width 0)
+			(type default)
+		)
+	)
+	(wire
+		(pts
 			(xy 177.8 166.37) (xy 181.61 166.37)
 		)
@@
 		)
 	)
+	(label "+5V-USB"
+		(at 48.26 55.88 180)
+		(effects
+			(font
+				(size 1.27 1.27)
+			)
+			(justify right bottom)
+		)
+	)
 	(label "ADC3_5"
 		(at 127 20.32 180)
@@
 		)
 	)
+	(label "+5V-JTAG"
+		(at 48.26 50.8 180)
+		(effects
+			(font
+				(size 1.27 1.27)
+			)
+			(justify right bottom)
+		)
+	)
 	(label "PD1"
 		(at 322.58 80.01 0)
@@
 		)
 	)
+	(label "+5V-JTAG"
+		(at 30.48 34.29 180)
+		(effects
+			(font
+				(size 1.27 1.27)
+			)
+			(justify right bottom)
+		)
+	)
+	(label "+5V-USB"
+		(at 40.64 80.01 180)
+		(effects
+			(font
+				(size 1.27 1.27)
+			)
+			(justify right bottom)
+		)
+	)
 	(label "PB3"
 		(at 266.7 83.82 0)
@@
 		)
 	)
-	(hierarchical_label "USB_FS_VBUS"
-		(shape bidirectional)
-		(at 40.64 80.01 180)
-		(effects
-			(font
-				(size 1.27 1.27)
-			)
-			(justify right)
-		)
-	)
 	(hierarchical_label "{UART2_TX UART2_RX}"
 		(shape bidirectional)
@@
 		)
 	)
+	(hierarchical_label "+5V"
+		(shape bidirectional)
+		(at 44.45 53.34 180)
+		(effects
+			(font
+				(size 1.27 1.27)
+			)
+			(justify right)
+		)
+	)
 	(hierarchical_label "~{nRST}"
 		(shape bidirectional)
@@
 	)
 	(symbol
-		(lib_id "power:+3.3V")
-		(at 35.56 34.29 90)
-		(unit 1)
-		(exclude_from_sim no)
-		(in_bom yes)
-		(on_board yes)
-		(dnp no)
-		(fields_autoplaced yes)
-		(property "Reference" "#PWR041"
-			(at 39.37 34.29 0)
-			(effects
-				(font
-					(size 1.27 1.27)
-				)
-				(hide yes)
-			)
-		)
-		(property "Value" "+3.3V"
-			(at 31.75 34.2899 90)
-			(effects
-				(font
-					(size 1.27 1.27)
-				)
-				(justify left)
-			)
-		)
-		(property "Footprint" ""
-			(at 35.56 34.29 0)
-			(effects
-				(font
-					(size 1.27 1.27)
-				)
-				(hide yes)
-			)
-		)
-		(property "Datasheet" ""
-			(at 35.56 34.29 0)
-			(effects
-				(font
-					(size 1.27 1.27)
-				)
-				(hide yes)
-			)
-		)
-		(property "Description" "Power symbol creates a global label with name \"+3.3V\""
-			(at 35.56 34.29 0)
-			(effects
-				(font
-					(size 1.27 1.27)
-				)
-				(hide yes)
-			)
-		)
-		(pin "1"
-		)
-		(instances
-			(project ""
-				(path "/bbb55367-1aa7-46ea-88d8-ce1ddc0fd963/868b9e21-e37c-4d93-baf9-b4839eaf8a01"
-					(reference "#PWR041")
-					(unit 1)
-				)
-			)
-		)
-	)
-	(symbol
 		(lib_id "power:VCC")
 		(at 223.52 96.52 90)
@@
 					(unit 1)
 				)
+			)
+		)
+	)
+	(symbol
+		(lib_id "Connector_Generic:Conn_01x03")
+		(at 53.34 53.34 0)
+		(unit 1)
+		(exclude_from_sim no)
+		(in_bom yes)
+		(on_board yes)
+		(dnp no)
+		(fields_autoplaced yes)
+		(property "Reference" "J12"
+			(at 55.88 52.0699 0)
+			(effects
+				(font
+					(size 1.27 1.27)
+				)
+				(justify left)
+			)
+		)
+		(property "Value" "Conn_01x03"
+			(at 55.88 54.6099 0)
+			(effects
+				(font
+					(size 1.27 1.27)
+				)
+				(justify left)
+			)
+		)
+		(property "Footprint" "Connector_PinHeader_2.54mm:PinHeader_1x03_P2.54mm_Vertical"
+			(at 53.34 53.34 0)
+			(effects
+				(font
+					(size 1.27 1.27)
+				)
+				(hide yes)
+			)
+		)
+		(property "Datasheet" "~"
+			(at 53.34 53.34 0)
+			(effects
+				(font
+					(size 1.27 1.27)
+				)
+				(hide yes)
+			)
+		)
+		(property "Description" "Generic connector, single row, 01x03, script generated (kicad-library-utils/schlib/autogen/connector/)"
+			(at 53.34 53.34 0)
+			(effects
+				(font
+					(size 1.27 1.27)
+				)
+				(hide yes)
+			)
+		)
+		(pin "2"
+		)
+		(pin "1"
+		)
+		(pin "3"
+		)
+		(instances
+			(project ""
+				(path "/bbb55367-1aa7-46ea-88d8-ce1ddc0fd963/868b9e21-e37c-4d93-baf9-b4839eaf8a01"
+					(reference "J12")
+					(unit 1)
+				)

Commit message: Final Updated design
Parts:
- renumbered J9 to J11, J6 to J3, J3 to J5, J5 to J6, J8 to J7, J7 to J8, J11 to J9
Connections:
- net PWM10 renamed PWM4
- net PWM11 renamed PWM5

Commit message: final submission
Connections:
- net GND: no longer J5.10
- new net GNDA: J5.10
