File: hardware/SimsBharath_DAQ_MCU.kicad_sch (KiCad schematic)
At the start: 40 parts, among them IC1 STM32H753ZIT6, IC2 MIC37100-3.3WS, Y1 XRCGB25M000F3A16R0, Y3 CM7V-T1A-32.768KHZ-7PF-20PPM-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

Commit message: updated
Parts:
- added +3.3V1, +5V1: TestPoint, TestPoint:TestPoint_Pad_D1.5mm, symbol Connector:TestPoint
- added C40: 0.1uF, Murata:GRM18x, symbol Murata:GRM188R72A104KA35D
- added R38, R39: 10k, Murata:RESC1608X95N, symbol Murata:PRF18BC471QB5RB
- added SW1: SW_Push, Button_Switch_THT:SW_PUSH_6mm_H4.3mm, symbol Switch:SW_Push
- renumbered IC1 to U1, IC2 to U2, Y1 to X1, Y3 to X3
Connections:
- net +3.3V: now also R3.2, +3.3V1.1, R38.2; no longer R3.1
- net +5V: now also +5V1.1
- net GND: now also C40.2, R39.2, SW1.2
- net VBAT: now also R3.1; no longer R3.2
- net ~{nRST}: now also C40.1, SW1.1
- net at U1.143 (PDR_ON): now also R38.1, R39.1
- no-connect marks 32 -> 31

Commit message: completed the design
Connections:
- net USB_FS_DM renamed USB_FS_D N
- net USB_FS_DP renamed USB_FS_D P
Changed lines of the file:
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@@
 	)
 	(bus_entry
-		(at 387.35 96.52)
-		(size 2.54 2.54)
-		(stroke
-			(width 0)
-			(type default)
-		)
-	)
-	(bus_entry
 		(at 373.38 129.54)
 		(size -2.54 2.54)
@@
 	)
 	(bus_entry
-		(at 387.35 96.52)
-		(size -2.54 2.54)
-		(stroke
-			(width 0)
-			(type default)
-		)
-	)
-	(bus_entry
 		(at 262.89 204.47)
 		(size 2.54 -2.54)
@@
 	)
 	(bus_entry
-		(at 387.35 93.98)
-		(size -2.54 2.54)
-		(stroke
-			(width 0)
-			(type default)
-		)
-	)
-	(bus_entry
 		(at 373.38 139.7)
 		(size -2.54 2.54)
@@
 	(wire
 		(pts
-			(xy 354.33 99.06) (xy 384.81 99.06)
-		)
-		(stroke
-			(width 0)
-			(type default)
-		)
-	)
-	(wire
-		(pts
 			(xy 270.51 55.88) (xy 270.51 68.58)
 		)
@@
 		)
 	)
+	(wire
+		(pts
+			(xy 354.33 99.06) (xy 359.41 99.06)
+		)
+		(stroke
+			(width 0)
+			(type default)
+		)
+	)
 	(bus
 		(pts
@@
 		)
 	)
-	(wire
-		(pts
-			(xy 354.33 96.52) (xy 384.81 96.52)
-		)
-		(stroke
-			(width 0)
-			(type default)
-		)
-	)
 	(bus
 		(pts
@@
 		)
 	)
-	(bus
-		(pts
-			(xy 387.35 93.98) (xy 387.35 96.52)
-		)
-		(stroke
-			(width 0)
-			(type default)
-		)
-	)
 	(wire
 		(pts
@@
 	(wire
 		(pts
+			(xy 354.33 96.52) (xy 359.41 96.52)
+		)
+		(stroke
+			(width 0)
+			(type default)
+		)
+	)
+	(wire
+		(pts
 			(xy 316.23 193.04) (xy 316.23 207.01)
 		)
@@
 		)
 	)
-	(wire
-		(pts
-			(xy 389.89 99.06) (xy 391.16 99.06)
-		)
-		(stroke
-			(width 0)
-			(type default)
-		)
-	)
 	(bus
 		(pts
@@
 		)
 	)
-	(bus
-		(pts
-			(xy 387.35 91.44) (xy 387.35 93.98)
-		)
-		(stroke
-			(width 0)
-			(type default)
-		)
-	)
 	(wire
 		(pts
@@
 	(wire
 		(pts
-			(xy 391.16 95.25) (xy 391.16 99.06)
-		)
-		(stroke
-			(width 0)
-			(type default)
-		)
-	)
-	(wire
-		(pts
 			(xy 190.5 71.12) (xy 190.5 72.39)
 		)
@@
 		)
 	)
-	(wire
-		(pts
-			(xy 392.43 93.98) (xy 391.16 95.25)
-		)
-		(stroke
-			(width 0)
-			(type default)
-		)
-	)
 	(bus
 		(pts
@@
 		)
 	)
-	(label "USB_FS_DP"
-		(at 354.33 96.52 0)
-		(effects
-			(font
-				(size 1.27 1.27)
-			)
-			(justify left bottom)
-		)
-	)
 	(label "UART1_RX"
 		(at 341.63 203.2 90)
@@
 		)
 	)
-	(label "USB_FS_VBUS"
-		(at 391.16 99.06 0)
-		(effects
-			(font
-				(size 1.27 1.27)
-			)
-			(justify left bottom)
-		)
-	)
 	(label "PD1"
 		(at 354.33 152.4 0)
@@
 		)
 	)
-	(label "USB_FS_DM"
-		(at 354.33 99.06 0)
-		(effects
-			(font
-				(size 1.27 1.27)
-			)
-			(justify left bottom)
-		)
-	)
 	(label "OSC32_IN"
 		(at 72.39 158.75 0)
@@
 		)
 	)
-	(hierarchical_label "{USB_FS_VBUS USB_FS_DM USB_FS_DP}"
-		(shape bidirectional)
-		(at 387.35 91.44 90)
-		(effects
-			(font
-				(size 1.27 1.27)
-			)
-			(justify left)
-		)
-	)
 	(hierarchical_label "ETH_RMII_RXD1"
 		(shape bidirectional)
@@
 		)
 	)
+	(hierarchical_label "USB_FS_D P"
+		(shape bidirectional)
+		(at 359.41 96.52 0)
+		(effects
+			(font
+				(size 1.27 1.27)
+			)
+			(justify left)
+		)
+	)
+	(hierarchical_label "USB_FS_D N"
+		(shape bidirectional)
+		(at 359.41 99.06 0)
+		(effects
+			(font
+				(size 1.27 1.27)
+			)
+			(justify left)
+		)
+	)
+	(hierarchical_label "USB_FS_VBUS"
+		(shape bidirectional)
+		(at 392.43 93.98 180)
+		(effects
+			(font
+				(size 1.27 1.27)
+			)
+			(justify right)
+		)
+	)

Commit message: completed the design with perfect mechanics
Changed lines of the file:
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@@
 	)
 	(junction
-		(at 398.78 90.17)
-		(diameter 0)
-		(color 0 0 0 0)
-	)
-	(junction
 		(at 40.64 119.38)
 		(diameter 0)
@@
 	(wire
 		(pts
-			(xy 398.78 93.98) (xy 398.78 90.17)
-		)
-		(stroke
-			(width 0)
-			(type default)
-		)
-	)
-	(wire
-		(pts
 			(xy 195.58 186.69) (xy 195.58 184.15)
 		)
@@
 	(wire
 		(pts
-			(xy 78.74 66.04) (xy 81.28 66.04)
+			(xy 78.74 66.04) (xy 87.63 66.04)
 		)
 		(stroke
@@
 	(wire
 		(pts
-			(xy 398.78 93.98) (xy 392.43 93.98)
-		)
-		(stroke
-			(width 0)
-			(type default)
-		)
-	)
-	(wire
-		(pts
 			(xy 210.82 167.64) (xy 215.9 167.64)
 		)
@@
 		)
 	)
-	(hierarchical_label "USB_FS_VBUS"
-		(shape bidirectional)
-		(at 392.43 93.98 180)
-		(effects
-			(font
-				(size 1.27 1.27)
-			)
-			(justify right)
-		)
-	)
 	(hierarchical_label "ETH_RMII_TX_EN"
 		(shape bidirectional)
@@
 	(symbol
 		(lib_id "power:+3.3V")
-		(at 81.28 66.04 270)
+		(at 87.63 66.04 270)
 		(unit 1)
 		(exclude_from_sim no)
@@
 		(dnp no)
 		(property "Reference" "#PWR045"
-			(at 77.47 66.04 0)
+			(at 83.82 66.04 0)
 			(effects
 				(font
@@
 		)
 		(property "Value" "+5V"
-			(at 84.328 66.04 90)
+			(at 90.678 66.04 90)
 			(effects
 				(font
@@
 		)
 		(property "Footprint" ""
-			(at 81.28 66.04 0)
+			(at 87.63 66.04 0)
 			(effects
 				(font
@@
 		)
 		(property "Datasheet" ""
-			(at 81.28 66.04 0)
+			(at 87.63 66.04 0)
 			(effects
 				(font
@@
 		)
 		(property "Description" "Power symbol creates a global label with name \"+3.3V\""
-			(at 81.28 66.04 0)
+			(at 87.63 66.04 0)
 			(effects
 				(font

Commit message: Final Updated design
Parts:
- added R40: 10k, Murata:RESC1608X95N, symbol Murata:PRF18BC471QB5RB
Connections:
- net PWM10 is gone; now on net PWM2: U1.60 (PE9)
- net GND: now also R40.2
- net PB4: now also U1.137 (PB7); no longer U1.138 (BOOT0)
- net PB5: now also U1.136 (PB6); no longer U1.137 (PB7)
- net PB6: now also U1.135 (PB5); no longer U1.136 (PB6)
- net PB7: now also U1.132 (PG15); no longer U1.135 (PB5)
- net PWM0: now also U1.97 (PC7); no longer U1.96 (PC6)
- net PWM1: now also U1.96 (PC6); no longer U1.97 (PC7)
- net PWM2: no longer U1.98 (PC8)
- net PWM3: now also U1.42 (PA6); no longer U1.99 (PC9)
- net SPI4_MISO: now also U1.4 (PE5); no longer U1.3 (PE4)
- net SPI4_MOSI: now also U1.5 (PE6); no longer U1.4 (PE5)
- net SPI4_NSS: now also U1.3 (PE4); no longer U1.2 (PE3)
- net SPI5_MOSI: now also U1.113 (PC12); no longer U1.111 (PC10)
- net SPI5_NSS: now also U1.114 (PD0); no longer U1.113 (PC12)
- net SPI5_SCK: now also U1.111 (PC10); no longer U1.114 (PD0)
- net PWM5: now reaches U1.34 (PA0-WKUP)
- net PWM4: now reaches U1.37 (PA3)
- net PWM11: no longer names the net of U1.64 (PE11)
- new net: R40.1, U1.138 (BOOT0)
- no-connect marks 31 -> 30

Commit message: final submission
Connections:
- net GNDA is gone; now on net GND: C15.2, C16.2, C17.2, C18.2, U1.31 (VSSA)
Changed lines of the file:
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@@
 	(wire
 		(pts
+			(xy 128.27 265.43) (xy 137.16 265.43)
+		)
+		(stroke
+			(width 0)
+			(type default)
+		)
+	)
+	(wire
+		(pts
 			(xy 303.53 193.04) (xy 303.53 207.01)
 		)
@@
 	)
 	(symbol
+		(lib_id "power:GND")
+		(at 137.16 265.43 0)
+		(unit 1)
+		(exclude_from_sim no)
+		(in_bom yes)
+		(on_board yes)
+		(dnp no)
+		(fields_autoplaced yes)
+		(property "Reference" "#PWR0102"
+			(at 137.16 271.78 0)
+			(effects
+				(font
+					(size 1.27 1.27)
+				)
+				(hide yes)
+			)
+		)
+		(property "Value" "GNDA"
+			(at 137.16 270.51 0)
+			(effects
+				(font
+					(size 1.27 1.27)
+				)
+			)
+		)
+		(property "Footprint" ""
+			(at 137.16 265.43 0)
+			(effects
+				(font
+					(size 1.27 1.27)
+				)
+				(hide yes)
+			)
+		)
+		(property "Datasheet" ""
+			(at 137.16 265.43 0)
+			(effects
+				(font
+					(size 1.27 1.27)
+				)
+				(hide yes)
+			)
+		)
+		(property "Description" "Power symbol creates a global label with name \"GND\" , ground"
+			(at 137.16 265.43 0)
+			(effects
+				(font
+					(size 1.27 1.27)
+				)
+				(hide yes)
+			)
+		)
+		(pin "1"
+		)
+		(instances
+			(project "SimsBharath_DAQ"
+				(path "/bbb55367-1aa7-46ea-88d8-ce1ddc0fd963/00b9c292-f450-48ac-8b34-fee93c972b1e"
+					(reference "#PWR0102")
+					(unit 1)
+				)
+			)
+		)
+	)
+	(symbol
 		(lib_id "Murata:GRM188R72A104KA35D")
 		(at 55.88 246.38 270)
@@
 					(unit 1)
 				)
+			)
+		)
+	)
+	(symbol
+		(lib_id "power:GND")
+		(at 128.27 265.43 0)
+		(unit 1)
+		(exclude_from_sim no)
+		(in_bom yes)
+		(on_board yes)
+		(dnp no)
+		(fields_autoplaced yes)
+		(property "Reference" "#PWR0101"
+			(at 128.27 271.78 0)
+			(effects
+				(font
+					(size 1.27 1.27)
+				)
+				(hide yes)
+			)
+		)
+		(property "Value" "GND"
+			(at 128.27 270.51 0)
+			(effects
+				(font
+					(size 1.27 1.27)
+				)
+			)
+		)
+		(property "Footprint" ""
+			(at 128.27 265.43 0)
+			(effects
+				(font
+					(size 1.27 1.27)
+				)
+				(hide yes)
+			)
+		)
+		(property "Datasheet" ""
+			(at 128.27 265.43 0)
+			(effects
+				(font
+					(size 1.27 1.27)
+				)
+				(hide yes)
+			)
+		)
+		(property "Description" "Power symbol creates a global label with name \"GND\" , ground"
+			(at 128.27 265.43 0)
+			(effects
+				(font
+					(size 1.27 1.27)
+				)
+				(hide yes)
+			)
+		)
+		(pin "1"
+		)
+		(instances
+			(project "SimsBharath_DAQ"
+				(path "/bbb55367-1aa7-46ea-88d8-ce1ddc0fd963/00b9c292-f450-48ac-8b34-fee93c972b1e"
+					(reference "#PWR0101")
+					(unit 1)
+				)
